Commit message: Fix palm collision mesh, reduce joint velocities.

File: robotiq_3f_gripper_visualization/cfg/robotiq-3f-gripper_articulated_macro.xacro (robot description, xacro)
@@ -23,5 +23,5 @@
 			<collision>
 				<geometry>
-                                        <mesh filename="package://robotiq_3f_gripper_visualization/meshes/robotiq-3f-gripper_articulated/collision/palm.STL" />
+                                        <mesh filename="package://robotiq_3f_gripper_visualization/meshes/robotiq-3f-gripper_articulated/collision/palm_with_finger_cutouts.stl" />
 				</geometry>
 				<material name="yellow">
@@ -43,5 +43,6 @@
 			<axis xyz="0 1 0"/>
 			<origin xyz="-0.0455 0.0214 0.036" rpy="0 3.1416 -1.57"/>
-			<limit lower="-0.1784" upper="0.192" effort="100" velocity="100"/>
+			<limit lower="-0.1784" upper="0.192" effort="100" velocity="1.23"/>
+      <dynamics friction="0.1" damping="1.0" />
 		</joint>
 		<joint name="${prefix}palm_finger_2_joint" type="revolute">
@@ -50,5 +51,6 @@
 			<axis xyz="0 1 0"/>
 			<origin xyz="-0.0455 0.0214 -0.036" rpy="0 3.1416 -1.57"/>
-			<limit lower="-0.192" upper="0.1784" effort="100" velocity="100"/>
+			<limit lower="-0.192" upper="0.1784" effort="100" velocity="1.23"/>
+      <dynamics friction="0.1" damping="1.0" />
 		</joint>
 		<joint name="${prefix}palm_finger_middle_joint" type="fixed">
