Commit message: Reduce joint velocities (for gazebo).

File: robotiq_3f_gripper_visualization/cfg/robotiq-3f-gripper_finger_articulated_macro.xacro (robot description, xacro)
@@ -108,5 +108,7 @@
 			<axis xyz="0 0 1"/>
 			<origin xyz="0.020 0 0" rpy="0 0 0"/>
-			<limit lower="0.0495" upper="1.2218" effort="100" velocity="100"/>
+      <!-- fnh: velocity=100 is far too fast. We also want some damping for Gazebo -->
+			<limit lower="0.0495" upper="1.2218" effort="100" velocity="1.23"/>
+      <dynamics friction="0.1" damping="1"/>
 		</joint>
 		<joint name="${prefix}joint_2" type="revolute">
@@ -115,5 +117,6 @@
 			<axis xyz="0 0 1"/>
 			<origin xyz="0.050 -.028 0" rpy="0 0 -0.52"/>
-			<limit lower="0.0" upper="1.5708" effort="100" velocity="100"/>
+			<limit lower="0.0" upper="1.5708" effort="100" velocity="1.24"/>
+      <dynamics friction="0.1" damping="1"/>
 		</joint>
 		<joint name="${prefix}joint_3" type="revolute">
@@ -122,5 +125,6 @@
 			<axis xyz="0 0 1"/>
 			<origin xyz="0.039 0 0" rpy="0 0 0"/>
-			<limit lower="-1.2217" upper="-0.0523" effort="100" velocity="100"/>
+			<limit lower="-1.2217" upper="-0.0523" effort="100" velocity="1.25"/>
+      <dynamics friction="0.1" damping="1"/>
 		</joint>
 		<!-- end of joint list -->
