Commit message: digit only on the left finger

File: robotiq_2f_85_gripper_visualization/urdf/robotiq_arg2f_85_digit_model_macro.xacro (robot description, xacro)
@@ -94,4 +94,28 @@
         <geometry>
           <mesh filename="package://robotiq_2f_85_gripper_visualization/meshes/collision/robotiq_arg2f_85_inner_finger.dae" scale="0.001 0.001 0.001" />
+        </geometry>
+      </collision>
+    </link>
+  </xacro:macro>
+  <xacro:macro name="inner_finger_digit_adapter" params="prefix fingerprefix stroke">
+    <link name="${prefix}${fingerprefix}_inner_finger">
+      <inertial>
+        <origin xyz="0.000299999999999317 0.0160078233491243 -0.0136945669206257" rpy="0 0 0" />
+        <mass value="0.0104003125914103" />
+        <inertia ixx="2.71909453810972E-06" ixy="1.35402465472579E-21" ixz="-7.1817349065269E-22" iyy="7.69100314106116E-07" iyz="6.74715432769696E-07" izz="2.30315190420171E-06" />
+        </inertial>
+      <visual>
+        <origin xyz="0 0 0" rpy="0 0 0" />
+        <geometry>
+          <mesh filename="package://sr_digit_launch/meshes/digit/digit_adapter_edited.dae" scale="0.001 0.001 0.001"/>
+        </geometry>
+        <material name="">
+          <color rgba="0.1 0.1 0.1 1" />
+        </material>
+      </visual>
+      <collision>
+        <origin xyz="0 0 0" rpy="0 0 0" />
+        <geometry>
+          <mesh filename="package://sr_digit_launch/meshes/digit/digit_adapter_edited.dae" scale="0.001 0.001 0.001"/>
         </geometry>
       </collision>
@@ -131,5 +155,5 @@
     </inertial>
     <visual>
-    <origin xyz="0 0 0" rpy="0 0 -1.57079632679"/>
+    <origin xyz="0 0.0135  0.012" rpy="0 -1.57079632679 1.57079632679"/>
       <geometry>
 				<mesh filename="package://sr_digit_launch/meshes/digit/digit.STL" scale="1 1 1"/>
@@ -140,5 +164,5 @@
     </visual>
     <collision concave="yes">
-    <origin xyz="0 0 0" rpy="0  0 -1.57079632679"/>
+    <origin xyz="0 0.0135  0.012" rpy="0 -1.57079632679 1.57079632679"/>
       <geometry>
 				<mesh filename="package://sr_digit_launch/meshes/digit/digit.STL" scale="1 1 1"/>
@@ -163,6 +187,15 @@
       <axis xyz="1 0 0" />
       <limit lower="0" upper="0.8757" velocity="2.0" effort="1000" />
-      <mimic joint="${prefix}finger_joint" multiplier="1" offset="0" />
-    </joint>
+      <!-- <mimic joint="${prefix}finger_joint" multiplier="1" offset="0" /> -->
+    </joint>
+    <transmission name="${prefix}${fingerprefix}_inner_knuckle_joint_trans">
+      <type>transmission_interface/SimpleTransmission</type>
+      <joint name="${prefix}${fingerprefix}_inner_knuckle_joint">
+        <hardwareInterface>hardware_interface/PositionJointInterface</hardwareInterface>
+      </joint>
+      <actuator name="${prefix}${fingerprefix}_inner_knuckle_joint_motor">
+        <mechanicalReduction>1</mechanicalReduction>
+      </actuator>
+    </transmission>
   </xacro:macro>
   <xacro:macro name="inner_finger_joint" params="prefix fingerprefix">
@@ -172,7 +205,17 @@
       <child link="${prefix}${fingerprefix}_inner_finger" />
       <axis xyz="1 0 0" />
-      <limit lower="0" upper="0.8757" velocity="2.0" effort="1000" />
-      <mimic joint="${prefix}finger_joint" multiplier="-1" offset="0" />
-    </joint>
+      <!-- <limit lower="0" upper="0.8757" velocity="2.0" effort="1000" /> -->
+      <limit lower="-0.8757" upper="0" velocity="2.0" effort="1000" />
+      <!--<mimic joint="${prefix}finger_joint" multiplier="-1" offset="0" /> -->
+    </joint>
+    <transmission name="${prefix}${fingerprefix}_inner_finger_joint_trans">
+      <type>transmission_interface/SimpleTransmission</type>
+      <joint name="${prefix}${fingerprefix}_inner_finger_joint">
+        <hardwareInterface>hardware_interface/PositionJointInterface</hardwareInterface>
+      </joint>
+      <actuator name="${prefix}${fingerprefix}_inner_finger_joint_motor">
+        <mechanicalReduction>1</mechanicalReduction>
+      </actuator>
+    </transmission>
   </xacro:macro>
   <xacro:macro name="inner_finger_pad_joint" params="prefix fingerprefix">
@@ -186,10 +229,8 @@
   <!-- I set the joint to revolute so i can get it's contacts as a topic -->
   <xacro:macro name="digit_joint" params="prefix fingerprefix">
-    <joint name="${prefix}${fingerprefix}_digit_joint" type="revolute">
-      <origin xyz="0 -0.01 0.044" rpy="0 0 0"/>
+    <joint name="${prefix}${fingerprefix}_digit_joint" type="fixed">
+      <origin xyz="0 -0.01 0.034" rpy="0 0 0"/>
       <parent link="${prefix}${fingerprefix}_inner_finger" />
       <child link="${prefix}${fingerprefix}_digit" />
-      <axis xyz="0 0 1" />
-      <limit effort="0" lower="0" upper="0" velocity="0"/>
     </joint>
   </xacro:macro>
@@ -212,6 +253,15 @@
       <axis xyz="1 0 0" />
       <limit lower="0" upper="0.81" velocity="2.0" effort="1000" />
-      <mimic joint="${prefix}finger_joint" multiplier="1" offset="0" />
-    </joint>
+      <!--<mimic joint="${prefix}finger_joint" multiplier="1" offset="0" /> -->
+    </joint>
+    <transmission name="${prefix}right_outer_knuckle_joint_trans">
+      <type>transmission_interface/SimpleTransmission</type>
+      <joint name="${prefix}right_outer_knuckle_joint">
+        <hardwareInterface>hardware_interface/PositionJointInterface</hardwareInterface>
+      </joint>
+      <actuator name="${prefix}right_outer_knuckle_joint_motor">
+        <mechanicalReduction>1</mechanicalReduction>
+      </actuator>
+    </transmission>
     <xacro:finger_joints prefix="${prefix}" fingerprefix="right" reflect="-1.0"/>
   </xacro:macro>
@@ -223,4 +273,7 @@
     <xacro:finger_joint prefix="${prefix}"/>
     <xacro:right_outer_knuckle_joint prefix="${prefix}"/>
+    <!-- Digit only on the left finger -->
+    <xacro:digit prefix="${prefix}" fingerprefix="left"/>
+    <xacro:digit_joint prefix="${prefix}" fingerprefix="left"/>
     <xacro:robotiq_arg2f_transmission prefix="${prefix}"/>
   </xacro:macro>

File: robotiq_2f_85_gripper_visualization/urdf/robotiq_arg2f_85_model_macro.xacro (robot description, xacro)
@@ -158,4 +158,5 @@
       <child link="${prefix}${fingerprefix}_inner_finger" />
       <axis xyz="1 0 0" />
+      <!-- <limit lower="0" upper="0.8757" velocity="2.0" effort="1000" /> -->
       <limit lower="-0.8757" upper="0" velocity="2.0" effort="1000" />
       <!--<mimic joint="${prefix}finger_joint" multiplier="-1" offset="0" /> -->

File: robotiq_2f_85_gripper_visualization/urdf/robotiq_arg2f_digit.xacro (robot description, xacro)
@@ -33,12 +33,12 @@
     <xacro:inner_finger_joint prefix="${prefix}" fingerprefix="${fingerprefix}"/>
     <!-- <xacro:inner_finger_pad_joint prefix="${prefix}" fingerprefix="${fingerprefix}"/> -->
-    <xacro:digit_joint prefix="${prefix}" fingerprefix="${fingerprefix}"/>
+    <!--<xacro:digit_joint prefix="${prefix}" fingerprefix="${fingerprefix}"/> -->
   </xacro:macro>
   <xacro:macro name="finger_links" params="prefix fingerprefix stroke">
     <xacro:outer_knuckle prefix="${prefix}" fingerprefix="${fingerprefix}" stroke="${stroke}"/>
     <xacro:outer_finger prefix="${prefix}" fingerprefix="${fingerprefix}" stroke="${stroke}"/>
-    <xacro:inner_finger prefix="${prefix}" fingerprefix="${fingerprefix}" stroke="${stroke}"/>
+    <xacro:inner_finger_digit_adapter prefix="${prefix}" fingerprefix="${fingerprefix}" stroke="${stroke}"/>
     <!--  <xacro:inner_finger_pad prefix="${prefix}" fingerprefix="${fingerprefix}"/> -->
-    <xacro:digit prefix="${prefix}" fingerprefix="${fingerprefix}"/>
+    <!--<xacro:digit prefix="${prefix}" fingerprefix="${fingerprefix}"/>-->
     <xacro:inner_knuckle prefix="${prefix}" fingerprefix="${fingerprefix}" stroke="${stroke}"/>
   </xacro:macro>

Commit message: renamed older

File: robotiq_2f_85_gripper_visualization/urdf/robotiq_arg2f_85_digit_model_macro.xacro (robot description, xacro)
@@ -108,14 +108,14 @@
         <origin xyz="0 0 0" rpy="0 0 0" />
         <geometry>
-          <mesh filename="package://sr_digit_launch/meshes/digit/digit_adapter_edited.dae" scale="0.001 0.001 0.001"/>
-        </geometry>
-        <material name="">
-          <color rgba="0.1 0.1 0.1 1" />
-        </material>
-      </visual>
-      <collision>
-        <origin xyz="0 0 0" rpy="0 0 0" />
-        <geometry>
-          <mesh filename="package://sr_digit_launch/meshes/digit/digit_adapter_edited.dae" scale="0.001 0.001 0.001"/>
+          <mesh filename="package://digit_gazebo_launch/meshes/digit/digit_adapter_edited.dae" scale="0.001 0.001 0.001"/>
+        </geometry>
+        <material name="">
+          <color rgba="0.1 0.1 0.1 1" />
+        </material>
+      </visual>
+      <collision>
+        <origin xyz="0 0 0" rpy="0 0 0" />
+        <geometry>
+          <mesh filename="package://digit_gazebo_launch/meshes/digit/digit_adapter_edited.dae" scale="0.001 0.001 0.001"/>
         </geometry>
       </collision>
@@ -157,5 +157,5 @@
     <origin xyz="0 0.0135  0.012" rpy="0 -1.57079632679 1.57079632679"/>
       <geometry>
-				<mesh filename="package://sr_digit_launch/meshes/digit/digit.STL" scale="1 1 1"/>
+				<mesh filename="package://digit_gazebo_launch/meshes/digit/digit.STL" scale="1 1 1"/>
       </geometry>
       <material name="white">
@@ -166,5 +166,5 @@
     <origin xyz="0 0.0135  0.012" rpy="0 -1.57079632679 1.57079632679"/>
       <geometry>
-				<mesh filename="package://sr_digit_launch/meshes/digit/digit.STL" scale="1 1 1"/>
+				<mesh filename="package://digit_gazebo_launch/meshes/digit/digit.STL" scale="1 1 1"/>
       </geometry>
     </collision>

Commit message: table_added

File: robotiq_2f_85_gripper_visualization/urdf/robotiq_arg2f_85_digit_model_macro.xacro (robot description, xacro)
@@ -150,10 +150,10 @@
   <link concave="yes" name="${prefix}${fingerprefix}_digit">
     <inertial>
-      <origin rpy="0 0 0" xyz="0 0 0.0135"/>
+      <origin rpy="0 0 0" xyz="0 0 0"/>
        <mass value=".02"/>
        <inertia ixx="2.9875E-8" ixy="0" ixz="0" iyy="1.273E-8" iyz="0" izz="3.2025E-8"/>
     </inertial>
     <visual>
-    <origin xyz="0 0.0135  0.012" rpy="0 -1.57079632679 1.57079632679"/>
+    <origin xyz="0 0  0" rpy="0 -1.57079632679 1.57079632679"/>
       <geometry>
 				<mesh filename="package://digit_gazebo_launch/meshes/digit/digit.STL" scale="1 1 1"/>
@@ -164,5 +164,5 @@
     </visual>
     <collision concave="yes">
-    <origin xyz="0 0.0135  0.012" rpy="0 -1.57079632679 1.57079632679"/>
+    <origin xyz="0 0  0" rpy="0 -1.57079632679 1.57079632679"/>
       <geometry>
 				<mesh filename="package://digit_gazebo_launch/meshes/digit/digit.STL" scale="1 1 1"/>
@@ -230,7 +230,14 @@
   <xacro:macro name="digit_joint" params="prefix fingerprefix">
     <joint name="${prefix}${fingerprefix}_digit_joint" type="fixed">
-      <origin xyz="0 -0.01 0.034" rpy="0 0 0"/>
+      <origin xyz="0 0.002 0.0465" rpy="0 0 0"/>
       <parent link="${prefix}${fingerprefix}_inner_finger" />
       <child link="${prefix}${fingerprefix}_digit" />
+    </joint>
+    <link name="digit_link">
+    </link>
+        <joint name="digit_link_joint" type="fixed">
+      <origin xyz="0 -0.018 0.06" rpy="0 -1.57079632679 1.57079632679"/>
+      <parent link="${prefix}${fingerprefix}_digit" />
+      <child link="digit_link" />
     </joint>
   </xacro:macro>

Commit message: digit frame

File: robotiq_2f_85_gripper_visualization/urdf/robotiq_arg2f_85_digit_model_macro.xacro (robot description, xacro)
@@ -237,5 +237,5 @@
     </link>
         <joint name="digit_link_joint" type="fixed">
-      <origin xyz="0 -0.018 0.06" rpy="0 -1.57079632679 1.57079632679"/>
+      <origin xyz="0 0 0" rpy="0 -1.57079632679 1.57079632679"/>
       <parent link="${prefix}${fingerprefix}_digit" />
       <child link="digit_link" />
