Commit message: tacto

File: robotiq_2f_85_gripper_visualization/urdf/robotiq_digit_ur_table.urdf.xacro (robot description, xacro)
@@ -55,12 +55,12 @@
     <xacro:table_macro/>
     <joint name="world_to_table" type="fixed">
-    <parent link="world"/>
-    <child link="table"/>
-        <origin xyz="0.0 $(arg initial_y) $(arg initial_z)" rpy="0.0 0.0 $(arg initial_yaw)"/>
+        <parent link="world"/>
+        <child link="table"/>
+            <origin xyz="0.0 $(arg initial_y) $(arg initial_z)" rpy="0.0 0.0 $(arg initial_yaw)"/>
     </joint>
     <joint name="table_to_robot" type="fixed">
-    <parent link="table"/>
-    <child link="$(arg arm_prefix)_base_link"/>
-    <origin xyz="-0.5 0 0.63" rpy="0 0 0"/>
+        <parent link="table"/>
+        <child link="$(arg arm_prefix)_base_link"/>
+        <origin xyz="-0.5 0 0.63" rpy="0 0 0"/>
     </joint>
     <xacro:robotiq_ft300 parent="$(arg arm_prefix)_flange" prefix="">
