Commit message: 2 cams

File: robotiq_2f_85_gripper_visualization/urdf/robotiq_arg2f_85_ur5e_wrist_cam.xacro (robot description, xacro)
@@ -16,20 +16,24 @@
     <color rgba="1.0 1.0 1.0 1.0"/>
   </material>
-  <xacro:macro name="robotiq_wrist_camera" params="parent prefix ">
+  <xacro:macro name="robotiq_wrist_camera" params="parent cam_prefix visual_flag *origin">
     <xacro:property name="camera_link" value="0.05" /> <!-- Size of square 'camera' box -->
-    <link name="camera_link">
-        <collision>
-            <origin xyz="0 0 0" rpy="0 0 0"/>
-            <geometry>
-                <box size="${camera_link} ${camera_link} ${camera_link}"/>
-            </geometry>
-        </collision>
-        <visual>
-            <origin xyz="0 0 0" rpy="0 0 0"/>
-            <geometry>
-                <box size="${camera_link} ${camera_link} ${camera_link}"/>
-            </geometry>
-            <material name="grey"/>
-        </visual>
+    <link name="camera_link${cam_prefix}">
+        <xacro:if value="${visual_flag == 'true'}">
+            <collision>
+                <origin xyz="0 0 0" rpy="0 0 0"/>
+                <geometry>
+                    <box size="${camera_link} ${camera_link} ${camera_link}"/>
+                </geometry>
+            </collision>
+        </xacro:if>
+        <xacro:if value="${visual_flag == 'true'}">
+            <visual>
+                <origin xyz="0 0 0" rpy="0 0 0"/>
+                <geometry>
+                    <box size="${camera_link} ${camera_link} ${camera_link}"/>
+                </geometry>
+                <material name="grey"/>
+            </visual>
+        </xacro:if>
         <inertial>
             <mass value="1e-5" />
@@ -38,13 +42,13 @@
         </inertial>
     </link>
-    <joint name="camera_joint" type="fixed">
+    <joint name="camera_joint${cam_prefix}" type="fixed">
         <axis xyz="0 1 0" />
-        <origin xyz="-0.07 0 0.02" rpy="0 -1.1 0"/>
+        <xacro:insert_block name="origin"/>
         <parent link="${parent}"/>
-        <child link="camera_link"/>
+        <child link="camera_link${cam_prefix}"/>
     </joint>
 <!-- camera -->
-    <gazebo reference="camera_link">
-        <sensor type="camera" name="camera0">
+    <gazebo reference="camera_link${cam_prefix}">
+        <sensor type="camera" name="camera${cam_prefix}">
         <update_rate>30.0</update_rate>
         <camera>
@@ -72,6 +76,6 @@
             <alwaysOn>true</alwaysOn>
             <updateRate>0.0</updateRate>
-            <cameraName>cameras/camera0</cameraName>
-            <frameName>camera_link</frameName>
+            <cameraName>cameras/camera${cam_prefix}</cameraName>
+            <frameName>camera_link${cam_prefix}</frameName>
             <depthImageTopicName>depth/image_raw</depthImageTopicName>
             <pointCloudTopicName>depth/points</pointCloudTopicName>

File: robotiq_2f_85_gripper_visualization/urdf/robotiq_digit_ur_table_cam.urdf.xacro (robot description, xacro)
@@ -70,5 +70,9 @@
     <!-- Create the Robotiq wrist camera -->
     <xacro:include filename="$(find robotiq_2f_85_gripper_visualization)/urdf/robotiq_arg2f_85_ur5e_wrist_cam.xacro" />
-    <xacro:robotiq_wrist_camera parent="$(arg hand_prefix)robotiq_arg2f_base_link" prefix="$(arg hand_prefix)">
+    <xacro:robotiq_wrist_camera parent="$(arg hand_prefix)robotiq_arg2f_base_link" cam_prefix="_0" visual_flag="false">
+        <origin xyz="-0.07 0 0.02" rpy="0 -1.1 0"/>
+    </xacro:robotiq_wrist_camera>
+    <xacro:robotiq_wrist_camera parent="world" cam_prefix="_1" visual_flag="true">
+        <origin xyz="0.6 0 1.5" rpy="${pi} ${3*pi/4} 0"/>
     </xacro:robotiq_wrist_camera>
     <!-- Create the Robotiq 2F-85 gripper -->

Commit message: cam

File: robotiq_2f_85_gripper_visualization/urdf/robotiq_arg2f_85_ur5e_wrist_cam.xacro (robot description, xacro)
@@ -19,5 +19,5 @@
     <xacro:property name="camera_link" value="0.05" /> <!-- Size of square 'camera' box -->
     <link name="camera_link${cam_prefix}">
-        <xacro:if value="${visual_flag == 'true'}">
+        <xacro:if value="${visual_flag}">
             <collision>
                 <origin xyz="0 0 0" rpy="0 0 0"/>
@@ -26,6 +26,4 @@
                 </geometry>
             </collision>
-        </xacro:if>
-        <xacro:if value="${visual_flag == 'true'}">
             <visual>
                 <origin xyz="0 0 0" rpy="0 0 0"/>

File: robotiq_2f_85_gripper_visualization/urdf/robotiq_digit_ur_table.urdf.xacro (robot description, xacro)
@@ -65,5 +65,5 @@
     </joint>
     <xacro:robotiq_ft300 parent="$(arg arm_prefix)_flange" prefix="">
-      <origin xyz="-0.005 0.0 0.0" rpy="${pi/2.0} ${pi/2.0} ${pi/2.0}"/>
+        <origin xyz="-0.005 0.0 0.0" rpy="${pi/2.0} ${pi/2.0} ${pi/2.0}"/>
     </xacro:robotiq_ft300>
     <xacro:robotiq_arg2f_85 prefix="$(arg hand_prefix)"/>

File: robotiq_2f_85_gripper_visualization/urdf/robotiq_digit_ur_table_cam.urdf.xacro (robot description, xacro)
@@ -70,5 +70,5 @@
     <!-- Create the Robotiq wrist camera -->
     <xacro:include filename="$(find robotiq_2f_85_gripper_visualization)/urdf/robotiq_arg2f_85_ur5e_wrist_cam.xacro" />
-    <xacro:robotiq_wrist_camera parent="$(arg hand_prefix)robotiq_arg2f_base_link" cam_prefix="_0" visual_flag="false">
+    <xacro:robotiq_wrist_camera parent="ft300_mounting_plate" cam_prefix="_0" visual_flag="true">
         <origin xyz="-0.07 0 0.02" rpy="0 -1.1 0"/>
     </xacro:robotiq_wrist_camera>
@@ -82,5 +82,5 @@
         <child link="$(arg hand_prefix)robotiq_arg2f_base_link"/>
         <origin xyz="0.0 0.0 0.0" rpy="0 ${pi} 0"/>
-    </joint>
+    </joint>y
     <gazebo reference="ra_wrist_3_joint">
         <provideFeedback>true</provideFeedback>
