Commit message: camera

File: robotiq_2f_85_gripper_visualization/urdf/robotiq_digit_ur_table_cam.urdf.xacro (robot description, xacro)
@@ -25,7 +25,7 @@
 -->
 <robot xmlns:xacro="http://www.ros.org/wiki/xacro"
-       xmlns:sensor="http://playerstage.sourceforge.net/gazebo/xmlschema/#sensor"
-       xmlns:controller="http://playerstage.sourceforge.net/gazebo/xmlschema/#controller"
-       xmlns:interface="http://playerstage.sourceforge.net/gazebo/xmlschema/#interface" name="urrobotiq">
+    xmlns:sensor="http://playerstage.sourceforge.net/gazebo/xmlschema/#sensor"
+    xmlns:controller="http://playerstage.sourceforge.net/gazebo/xmlschema/#controller"
+    xmlns:interface="http://playerstage.sourceforge.net/gazebo/xmlschema/#interface" name="urrobotiq">
     <link name="world"/>
     <xacro:arg name="initial_y" default="0.0"/>
@@ -65,5 +65,5 @@
     </joint>
     <xacro:robotiq_ft300 parent="$(arg arm_prefix)_flange" prefix="">
-      <origin xyz="-0.005 0.0 0.0" rpy="${pi/2.0} ${pi/2.0} ${pi/2.0}"/>
+        <origin xyz="-0.005 0.0 0.0" rpy="${pi/2.0} ${pi/2.0} ${pi/2.0}"/>
     </xacro:robotiq_ft300>
     <!-- Camera -->
