Commit message: joint name adjusted

File: robotiq_ft_sensor/urdf/robotiq_ft300.urdf.xacro (robot description, xacro)
@@ -61,6 +61,7 @@
             </collision>
         </link>
-         <!-- Connect force sensor with mounting/coupling plate -->
-        <joint name="${prefix}ft300_mounting_plate" type="fixed">
+        <!-- Connect force sensor with mounting/coupling plate -->
+        <!-- changed name from ft300_mounting_plate to ft300_mounting_plate_joint since it hase the same name as the link -->
+        <joint name="${prefix}ft300_mounting_plate_joint" type="fixed">
             <origin xyz="0 0 0.0415" rpy="0 ${pi} 0"/>
             <parent link="${prefix}ft300_mounting_plate" />
